File: 625nm/basic_led.kicad_pcb (KiCad board)
At the start: 2 copper layers, 25.4 x 20 mm, 8 parts, among them J1 Conn_01x04, J2 Conn_01x04, M1 MountingHole_2.5mm_Pad, M2 MountingHole_2.5mm_Pad, M3 MountingHole_2.5mm_Pad, M4 MountingHole_2.5mm_Pad

Commit message: Changed wavelength text on red LED from 625 to 630.
Other:
- board text added: "Basic LED V0.1 R1 www.iorodeo.com λ = 630nm"
- board text removed: "Basic LED V0.1 R1 www.iorodeo.com λ = 625nm"
Changed lines of the file:
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@@
       (effects (font (size 1 1) (thickness 0.15)))
     )
+    (fp_line (start -3 1.695) (end -3 -2.655) (layer F.SilkS) (width 0.15))
+    (fp_line (start 3 1.695) (end -3 1.695) (layer F.SilkS) (width 0.15))
+    (fp_line (start 3 -2.655) (end 3 1.695) (layer F.SilkS) (width 0.15))
+    (fp_line (start 0 -2.655) (end -3 -2.655) (layer F.SilkS) (width 0.15))
     (fp_line (start 3 -2.655) (end 0 -2.655) (layer F.SilkS) (width 0.15))
-    (fp_line (start 0 -2.655) (end -3 -2.655) (layer F.SilkS) (width 0.15))
-    (fp_line (start 3 -2.655) (end 3 1.695) (layer F.SilkS) (width 0.15))
-    (fp_line (start 3 1.695) (end -3 1.695) (layer F.SilkS) (width 0.15))
-    (fp_line (start -3 1.695) (end -3 -2.655) (layer F.SilkS) (width 0.15))
     (pad "" smd rect (at -2.65 -0.48 90) (size 0.8 3) (layers F.Cu F.Paste F.Mask))
     (pad "" smd rect (at 2.65 -0.48 90) (size 0.8 3) (layers F.Cu F.Paste F.Mask))
@@
       (effects (font (size 1 1) (thickness 0.15)))
     )
+    (fp_line (start -3 1.695) (end -3 -2.655) (layer F.SilkS) (width 0.15))
+    (fp_line (start 3 1.695) (end -3 1.695) (layer F.SilkS) (width 0.15))
+    (fp_line (start 3 -2.655) (end 3 1.695) (layer F.SilkS) (width 0.15))
+    (fp_line (start 0 -2.655) (end -3 -2.655) (layer F.SilkS) (width 0.15))
     (fp_line (start 3 -2.655) (end 0 -2.655) (layer F.SilkS) (width 0.15))
-    (fp_line (start 0 -2.655) (end -3 -2.655) (layer F.SilkS) (width 0.15))
-    (fp_line (start 3 -2.655) (end 3 1.695) (layer F.SilkS) (width 0.15))
-    (fp_line (start 3 1.695) (end -3 1.695) (layer F.SilkS) (width 0.15))
-    (fp_line (start -3 1.695) (end -3 -2.655) (layer F.SilkS) (width 0.15))
     (pad "" smd rect (at -2.65 -0.48 270) (size 0.8 3) (layers F.Cu F.Paste F.Mask))
     (pad "" smd rect (at 2.65 -0.48 270) (size 0.8 3) (layers F.Cu F.Paste F.Mask))
@@
       (effects (font (size 1 1) (thickness 0.15)))
     )
-    (fp_circle (center 0 0) (end 2.45 0) (layer F.SilkS) (width 0.15))
-    (fp_circle (center 0 0) (end 1.9 0) (layer F.SilkS) (width 0.05))
-    (fp_circle (center 0 0) (end 2.45 0) (layer B.SilkS) (width 0.15))
+    (fp_circle (center 0 0) (end 2.45 0) (layer B.SilkS) (width 0.15))
+    (fp_circle (center 0 0) (end 1.9 0) (layer F.SilkS) (width 0.05))
+    (fp_circle (center 0 0) (end 2.45 0) (layer F.SilkS) (width 0.15))
     (fp_text user %R (at 0.3 0) (layer F.Fab) hide
       (effects (font (size 0.8 0.8) (thickness 0.16)))
@@
       (effects (font (size 1 1) (thickness 0.15)))
     )
-    (fp_circle (center 0 0) (end 2.45 0) (layer F.SilkS) (width 0.15))
-    (fp_circle (center 0 0) (end 1.9 0) (layer F.SilkS) (width 0.05))
-    (fp_circle (center 0 0) (end 2.45 0) (layer B.SilkS) (width 0.15))
+    (fp_circle (center 0 0) (end 2.45 0) (layer B.SilkS) (width 0.15))
+    (fp_circle (center 0 0) (end 1.9 0) (layer F.SilkS) (width 0.05))
+    (fp_circle (center 0 0) (end 2.45 0) (layer F.SilkS) (width 0.15))
     (fp_text user %R (at 0.3 0) (layer F.Fab) hide
       (effects (font (size 0.8 0.8) (thickness 0.16)))
@@
       (effects (font (size 1 1) (thickness 0.15)))
     )
-    (fp_circle (center 0 0) (end 2.45 0) (layer F.SilkS) (width 0.15))
-    (fp_circle (center 0 0) (end 1.9 0) (layer F.SilkS) (width 0.05))
-    (fp_circle (center 0 0) (end 2.45 0) (layer B.SilkS) (width 0.15))
+    (fp_circle (center 0 0) (end 2.45 0) (layer B.SilkS) (width 0.15))
+    (fp_circle (center 0 0) (end 1.9 0) (layer F.SilkS) (width 0.05))
+    (fp_circle (center 0 0) (end 2.45 0) (layer F.SilkS) (width 0.15))
     (fp_text user %R (at 0.3 0) (layer F.Fab) hide
       (effects (font (size 0.8 0.8) (thickness 0.16)))
@@
       (effects (font (size 1 1) (thickness 0.15)))
     )
-    (fp_circle (center 0 0) (end 2.45 0) (layer F.SilkS) (width 0.15))
-    (fp_circle (center 0 0) (end 1.9 0) (layer F.SilkS) (width 0.05))
-    (fp_circle (center 0 0) (end 2.45 0) (layer B.SilkS) (width 0.15))
+    (fp_circle (center 0 0) (end 2.45 0) (layer B.SilkS) (width 0.15))
+    (fp_circle (center 0 0) (end 1.9 0) (layer F.SilkS) (width 0.05))
+    (fp_circle (center 0 0) (end 2.45 0) (layer F.SilkS) (width 0.15))
     (fp_text user %R (at 0.3 0) (layer F.Fab) hide
       (effects (font (size 0.8 0.8) (thickness 0.16)))
@@
       (effects (font (size 1 1) (thickness 0.15)))
     )
+    (fp_line (start 1.48 0.73) (end -1.48 0.73) (layer F.CrtYd) (width 0.05))
+    (fp_line (start 1.48 -0.73) (end 1.48 0.73) (layer F.CrtYd) (width 0.05))
+    (fp_line (start -1.48 -0.73) (end 1.48 -0.73) (layer F.CrtYd) (width 0.05))
+    (fp_line (start -1.48 0.73) (end -1.48 -0.73) (layer F.CrtYd) (width 0.05))
+    (fp_line (start -1.485 0.735) (end 0.8 0.735) (layer F.SilkS) (width 0.12))
+    (fp_line (start -1.485 -0.735) (end -1.485 0.735) (layer F.SilkS) (width 0.12))
+    (fp_line (start 0.8 -0.735) (end -1.485 -0.735) (layer F.SilkS) (width 0.12))
+    (fp_line (start 0.8 0.4) (end 0.8 -0.4) (layer F.Fab) (width 0.1))
+    (fp_line (start -0.8 0.4) (end 0.8 0.4) (layer F.Fab) (width 0.1))
+    (fp_line (start -0.8 -0.1) (end -0.8 0.4) (layer F.Fab) (width 0.1))
+    (fp_line (start -0.5 -0.4) (end -0.8 -0.1) (layer F.Fab) (width 0.1))
     (fp_line (start 0.8 -0.4) (end -0.5 -0.4) (layer F.Fab) (width 0.1))
-    (fp_line (start -0.5 -0.4) (end -0.8 -0.1) (layer F.Fab) (width 0.1))
-    (fp_line (start -0.8 -0.1) (end -0.8 0.4) (layer F.Fab) (width 0.1))
-    (fp_line (start -0.8 0.4) (end 0.8 0.4) (layer F.Fab) (width 0.1))
-    (fp_line (start 0.8 0.4) (end 0.8 -0.4) (layer F.Fab) (width 0.1))
-    (fp_line (start 0.8 -0.735) (end -1.485 -0.735) (layer F.SilkS) (width 0.12))
-    (fp_line (start -1.485 -0.735) (end -1.485 0.735) (layer F.SilkS) (width 0.12))
-    (fp_line (start -1.485 0.735) (end 0.8 0.735) (layer F.SilkS) (width 0.12))
-    (fp_line (start -1.48 0.73) (end -1.48 -0.73) (layer F.CrtYd) (width 0.05))
-    (fp_line (start -1.48 -0.73) (end 1.48 -0.73) (layer F.CrtYd) (width 0.05))
-    (fp_line (start 1.48 -0.73) (end 1.48 0.73) (layer F.CrtYd) (width 0.05))
-    (fp_line (start 1.48 0.73) (end -1.48 0.73) (layer F.CrtYd) (width 0.05))
     (fp_text user %R (at 0 0 90) (layer F.Fab)
       (effects (font (size 0.8 0.8) (thickness 0.16)))
@@
       (effects (font (size 0.8 0.8) (thickness 0.16)))
     )
+    (fp_line (start -0.8 0.4125) (end -0.8 -0.4125) (layer F.Fab) (width 0.1))
+    (fp_line (start -0.8 -0.4125) (end 0.8 -0.4125) (layer F.Fab) (width 0.1))
+    (fp_line (start 0.8 -0.4125) (end 0.8 0.4125) (layer F.Fab) (width 0.1))
+    (fp_line (start 0.8 0.4125) (end -0.8 0.4125) (layer F.Fab) (width 0.1))
+    (fp_line (start -0.237258 -0.5225) (end 0.237258 -0.5225) (layer F.SilkS) (width 0.12))
+    (fp_line (start -0.237258 0.5225) (end 0.237258 0.5225) (layer F.SilkS) (width 0.12))
+    (fp_line (start -1.48 0.73) (end -1.48 -0.73) (layer F.CrtYd) (width 0.05))
+    (fp_line (start -1.48 -0.73) (end 1.48 -0.73) (layer F.CrtYd) (width 0.05))
+    (fp_line (start 1.48 -0.73) (end 1.48 0.73) (layer F.CrtYd) (width 0.05))
     (fp_line (start 1.48 0.73) (end -1.48 0.73) (layer F.CrtYd) (width 0.05))
-    (fp_line (start 1.48 -0.73) (end 1.48 0.73) (layer F.CrtYd) (width 0.05))
-    (fp_line (start -1.48 -0.73) (end 1.48 -0.73) (layer F.CrtYd) (width 0.05))
-    (fp_line (start -1.48 0.73) (end -1.48 -0.73) (layer F.CrtYd) (width 0.05))
-    (fp_line (start -0.237258 0.5225) (end 0.237258 0.5225) (layer F.SilkS) (width 0.12))
-    (fp_line (start -0.237258 -0.5225) (end 0.237258 -0.5225) (layer F.SilkS) (width 0.12))
-    (fp_line (start 0.8 0.4125) (end -0.8 0.4125) (layer F.Fab) (width 0.1))
-    (fp_line (start 0.8 -0.4125) (end 0.8 0.4125) (layer F.Fab) (width 0.1))
-    (fp_line (start -0.8 -0.4125) (end 0.8 -0.4125) (layer F.Fab) (width 0.1))
-    (fp_line (start -0.8 0.4125) (end -0.8 -0.4125) (layer F.Fab) (width 0.1))
     (fp_text user %R (at 0 0) (layer F.Fab)
       (effects (font (size 0.4 0.4) (thickness 0.06)))
@@
     )
   )
-  (gr_text "Basic LED V0.1 R1\nwww.iorodeo.com\nλ = 625nm" (at 62.7 60) (layer B.SilkS)
+  (gr_text "Basic LED V0.1 R1\nwww.iorodeo.com\nλ = 630nm" (at 62.7 60) (layer B.SilkS)
     (effects (font (size 1 1) (thickness 0.15)) (justify mirror))
   )
