File: 625nm/basic_led.sch (KiCad schematic (older format))
At the start: 4 parts, among them J1 Conn_01x04, J2 Conn_01x04

Commit message: Changed wavelength text on red LED from 625 to 630.
Other:
- note added: "630nm LED (Vf=2V, I=16mA)"
- note removed: "625nm LED (Vf=2V, I=16mA)"
Changed lines of the file:
@@
 $EndComp
 Text Notes 3825 1000 0    50   ~ 0
-625nm LED (Vf=2V, I=16mA)
+630nm LED (Vf=2V, I=16mA)
 $EndSCHEMATC
